File: autopilotv1/autopilotv1.kicad_pcb (KiCad board)
At the start: 2 copper layers, 111 x 78 mm, 20 parts, among them J1 Conn_01x01, M3 MountingHole_3.2mm_M3_Pad, SW1 My2pin_SW_MEC_5G, SW10 My2pin_SW_MEC_5G, SW11 Rotary_Encoder_Switch, SW12 Rotary_Encoder_Switch, SW13 Rotary_Encoder_Switch, SW14 Rotary_Encoder_Switch, SW15 Rotary_Encoder_Switch, SW2 My2pin_SW_MEC_5G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

Commit message: It works!
Other:
- board text added: "JLCJLCJLCJLC"
